File: wi-se-rewirable/wi-se-rewirable.kicad_pcb (KiCad board)
At the start: 4 copper layers, 25.5 x 22.4 mm, 50 parts, among them J1 FLASHING, J2 REWIRABLE, Q1 SS8050-G, Q2 SS8050-G, SW1 RESET, SW2 BOOT0, U1 AMS1117-3.3, U2 ESP-WROOM-02

Commit message: rewirable: Add missing GPIO15 pull-down
Parts:
- added R14: 10k, Resistor_SMD:R_0402_1005Metric, B.Cu at (113.4, 85.4)
Connections:
- U2 pad 6: (no net) -> Net-(R14-Pad2)
Routing:
- net Net-(R14-Pad2): track 0.00 -> 2.99 mm, vias 0 -> 1
- net GND: track 98.7 -> 101.1 mm
Other:
- board text added: "v0.2 rewirable"
- board text removed: "v0.1 rewirable"
