File: wi-se-rewirable/wi-se-rewirable.sch (KiCad schematic (older format))
At the start: 50 parts, among them J1 FLASHING, J2 REWIRABLE, Q1 SS8050-G, Q2 SS8050-G, SW1 RESET, SW2 BOOT0, U1 AMS1117-3.3, U2 ESP-WROOM-02

Commit message: rewirable: Add missing GPIO15 pull-down
Parts:
- added R14: 10k, Resistor_SMD:R_0402_1005Metric, symbol Device:R_Small
Connections:
- wire segments 116 -> 118
- no-connect marks 5 -> 4
Changed lines of the file:
@@
 Text GLabel 9750 3650 2    50   Input ~ 0
 LED_STATUS
-NoConn ~ 9750 3850
 NoConn ~ 9750 3350
 NoConn ~ 8750 3450
@@
 Wire Wire Line
 	1500 1200 2950 1200
+$Comp
+L Device:R_Small R14
+U 1 1 6054FB47
+P 10000 3850
+F 0 "R14" V 10100 3850 50  0000 C CNN
+F 1 "10k" V 10200 3850 50  0000 C CNN
+F 2 "Resistor_SMD:R_0402_1005Metric" H 10000 3850 50  0001 C CNN
+F 3 "~" H 10000 3850 50  0001 C CNN
+F 4 "C25744" H 10000 3850 50  0001 C CNN "LCSC Part"
+	1    10000 3850
+	0    1    1    0
+$EndComp
+Wire Wire Line
+	9750 3850 9900 3850
+$Comp
+L power:GND #PWR01
+U 1 1 60555AD4
+P 10450 3850
+F 0 "#PWR01" H 10450 3600 50  0001 C CNN
+F 1 "GND" H 10455 3677 50  0000 C CNN
+F 2 "" H 10450 3850 50  0001 C CNN
+F 3 "" H 10450 3850 50  0001 C CNN
+	1    10450 3850
+	1    0    0    -1
+$EndComp
+Wire Wire Line
+	10450 3850 10100 3850
 $EndSCHEMATC
